File: USB-Breakout/USB-Breakout.kicad_pcb (KiCad board)
At the start: 2 copper layers, 25 x 25 mm, 16 parts, among them J1 Conn_02x07_Odd_Even, J2 12401951E412A, Q1 IRLZ44N, Q2 IRF4905, U1 FUSB302BMPX

Commit message: Update documentation and improve project structure for better usability
Routing:
- net +3.3V: track 38.7 -> 24.5 mm, vias 1 -> 2
- net +5V: track 22.3 -> 32.3 mm, vias 1 -> 0
- net /SCL: track 16.0 -> 7.11 mm
- net /D+: track 27.8 -> 33.2 mm
- net GND: track 6.44 -> 1.11 mm, vias 10 -> 4
- net /D-: track 29.0 -> 32.7 mm
- net /CC1: track 30.3 -> 32.7 mm, vias 3 -> 1
- net VBUS: track 50.4 -> 52.6 mm, vias 0 -> 2
- net /5_EN: track 26.7 -> 25.4 mm
- net /12_EN: track 12.3 -> 11.2 mm
- net /CC2: track 22.0 -> 20.9 mm, vias 1 -> 0
- net /SDA: track 5.32 -> 6.40 mm
- net /INT: track 8.61 -> 8.02 mm, vias 1 -> 0
- added copper zone on In1.Cu, net GND
- added copper zone on In2.Cu, net GND
Other:
- copper layers 2 -> 4

Commit message: confused now
Parts:
- C2, C5: footprint Capacitor_THT:CP_Radial_D12.5mm_P2.50mm -> Capacitor_THT:C_Rect_L9.0mm_W6.4mm_P7.50mm_MKT
Routing:
- net GND: track 1.11 -> 20.4 mm, vias 4 -> 8
- net VBUS: track 52.6 -> 47.4 mm, vias 2 -> 3
- net +5V: track 32.3 -> 29.9 mm, vias 0 -> 1
- net /CC2: track 20.9 -> 23.0 mm
- net /D-: track 32.7 -> 34.6 mm
- net +3.3V: track 24.5 -> 26.2 mm
- net +12V: track 13.1 -> 14.4 mm
- net /INT: track 8.02 -> 9.16 mm
- net /12_EN: track 11.2 -> 12.3 mm
- net /CC1: track 32.7 -> 32.0 mm
- net /5_EN: track 25.4 -> 24.9 mm
Other:
- board size 25 x 25 mm -> 32.6 x 25 mm
