File: USB-Breakout/USB-Breakout.kicad_sch (KiCad schematic)
At the start: 16 parts, among them J1 Conn_02x07_Odd_Even, J2 12401951E412A, Q1 IRLZ44N, Q2 IRF4905, U1 FUSB302BMPX

Commit message: confused now
Parts:
- C2, C5: footprint Capacitor_THT:CP_Radial_D12.5mm_P2.50mm -> Capacitor_THT:C_Rect_L9.0mm_W6.4mm_P7.50mm_MKT
Changed lines of the file:
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@@
 			)
 		)
-		(property "Footprint" "Capacitor_THT:CP_Radial_D12.5mm_P2.50mm"
+		(property "Footprint" "Capacitor_THT:C_Rect_L9.0mm_W6.4mm_P7.50mm_MKT"
 			(at 143.51 106.68 0)
 			(effects
@@
 			)
 		)
-		(property "Footprint" "Capacitor_THT:CP_Radial_D12.5mm_P2.50mm"
+		(property "Footprint" "Capacitor_THT:C_Rect_L9.0mm_W6.4mm_P7.50mm_MKT"
 			(at 162.56 106.68 0)
 			(effects
